File: zx81-external-eprom.kicad_sch (KiCad schematic)
At the start: 10 parts, among them J1 Connector ZX81, Q1 BC549, SW1 SW_DIP_x03, U1 W27C512, U2 74LS138

Commit message: small cosmetic changes
Other:
- company: (none) -> ZXINFO
- title: (none) -> ZX81 External EPROM interface
- moved on the sheet: R1, R2, R3, SW1

Commit message: Local SYMBOL & FOOTPRINT
Parts:
- J1: footprint ZXINFO:EDGE ZX81_1 -> ZXINFO_FOOTPRINT:EDGE ZX81 BOTTOM; symbol ZXINFO_LIB:Connector ZX81 -> ZXINFO_SYMBOL:Connector ZX81
- U1: symbol ZXINFO_LIB:W27C512 -> ZXINFO_SYMBOL:W27C512
Changed lines of the file:
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@@
 	)
 	(symbol
-		(lib_id "ZXINFO_LIB:W27C512")
+		(lib_id "ZXINFO_SYMBOL:W27C512")
 		(at 149.86 100.33 0)
 		(unit 1)
@@
 	)
 	(symbol
-		(lib_id "ZXINFO_LIB:Connector ZX81")
+		(lib_id "ZXINFO_SYMBOL:Connector ZX81")
 		(at 40.64 66.04 0)
 		(unit 1)
@@
 			)
 		)
-		(property "Footprint" "ZXINFO:EDGE ZX81_1"
+		(property "Footprint" "ZXINFO_FOOTPRINT:EDGE ZX81 BOTTOM"
 			(at 40.64 62.23 0)
 			(effects
@@
 					(size 1.27 1.27)
 				)
-				(hide yes)
-			)
-		)
+			)
+		)

Commit message: changed Resistor to 10K
Parts:
- R1, R2, R3: value 4K7 -> 10K
Connections:
- net at R3.1, U1.1 (A15): now also SW1.6; no longer SW1.4
- net at R1.1, U1.26 (A13): now also SW1.4; no longer SW1.6
Changed lines of the file:
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@@
 	)
 	(junction
+		(at 128.27 143.51)
+		(diameter 0)
+		(color 0 0 0 0)
+	)
+	(junction
 		(at 90.17 143.51)
 		(diameter 0)
@@
 	)
 	(junction
-		(at 133.35 143.51)
-		(diameter 0)
-		(color 0 0 0 0)
-	)
-	(junction
 		(at 128.27 156.21)
 		(diameter 0)
@@
 	)
 	(junction
-		(at 128.27 138.43)
+		(at 149.86 134.62)
 		(diameter 0)
 		(color 0 0 0 0)
 	)
 	(junction
-		(at 149.86 134.62)
+		(at 133.35 138.43)
 		(diameter 0)
 		(color 0 0 0 0)
@@
 	(wire
 		(pts
-			(xy 69.85 46.99) (xy 77.47 46.99)
+			(xy 128.27 143.51) (xy 128.27 148.59)
 		)
 		(stroke
@@
 	(wire
 		(pts
-			(xy 90.17 140.97) (xy 90.17 143.51)
+			(xy 111.76 138.43) (xy 133.35 138.43)
 		)
 		(stroke
@@
 	(wire
 		(pts
-			(xy 57.15 109.22) (xy 57.15 92.71)
+			(xy 69.85 46.99) (xy 77.47 46.99)
 		)
 		(stroke
@@
 	(wire
 		(pts
-			(xy 111.76 138.43) (xy 128.27 138.43)
+			(xy 90.17 140.97) (xy 90.17 143.51)
 		)
 		(stroke
@@
 	(wire
 		(pts
-			(xy 128.27 104.14) (xy 128.27 138.43)
+			(xy 57.15 109.22) (xy 57.15 92.71)
 		)
 		(stroke
@@
 	(wire
 		(pts
-			(xy 19.05 124.46) (xy 85.09 124.46)
+			(xy 128.27 104.14) (xy 128.27 143.51)
+		)
+		(stroke
+			(width 0)
+			(type default)
+		)
+	)
+	(wire
+		(pts
+			(xy 111.76 143.51) (xy 128.27 143.51)
 		)
 		(stroke
@@
 	(wire
 		(pts
-			(xy 133.35 143.51) (xy 133.35 148.59)
+			(xy 19.05 124.46) (xy 85.09 124.46)
 		)
 		(stroke
@@
 	(wire
 		(pts
-			(xy 133.35 109.22) (xy 133.35 143.51)
+			(xy 133.35 109.22) (xy 133.35 138.43)
 		)
 		(stroke
@@
 	(wire
 		(pts
-			(xy 111.76 143.51) (xy 133.35 143.51)
-		)
-		(stroke
-			(width 0)
-			(type default)
-		)
-	)
-	(wire
-		(pts
 			(xy 125.73 80.01) (xy 125.73 119.38)
 		)
@@
 	(wire
 		(pts
-			(xy 128.27 138.43) (xy 128.27 148.59)
+			(xy 40.64 116.84) (xy 81.28 116.84)
 		)
 		(stroke
@@
 	(wire
 		(pts
-			(xy 40.64 116.84) (xy 81.28 116.84)
+			(xy 57.15 46.99) (xy 69.85 46.99)
 		)
 		(stroke
@@
 	(wire
 		(pts
-			(xy 57.15 46.99) (xy 69.85 46.99)
+			(xy 133.35 138.43) (xy 133.35 148.59)
 		)
 		(stroke
@@
 		)
 	)
+	(text_box "ZX81 external multi ROM interface\n\n- Re-wire, A15 -> 1-6, A13 -> 3-4\n	(position DIP correct)\n- Change R from 4K7 to 10K"
+		(exclude_from_sim no)
+		(at 195.58 15.24 0)
+		(size 86.36 31.75)
+		(stroke
+			(width 0)
+			(type dash)
+		)
+		(fill
+			(type none)
+		)
+		(effects
+			(font
+				(size 2 2)
+			)
+			(justify left top)
+		)
+	)
 	(global_label "A14"
 		(shape input)
@@
 			)
 		)
-		(property "Value" "4K7"
+		(property "Value" "10K"
 			(at 128.27 154.178 90)
 			(effects
@@
 			)
 		)
-		(property "Value" "4K7"
+		(property "Value" "10K"
 			(at 133.35 154.178 90)
 			(effects
@@
 			)
 		)
-		(property "Value" "4K7"
+		(property "Value" "10K"
 			(at 130.81 154.178 90)
 			(effects

Commit message: version 1.2
Parts:
- removed SW1: SW_DIP_x03, Button_Switch_THT:SW_DIP_SPSTx03_Slide_6.7x9.18mm_W7.62mm_P2.54mm_LowProfile, symbol Switch:SW_DIP_x03
- added C3: 100nF, Capacitor_THT:C_Disc_D3.0mm_W1.6mm_P2.50mm, symbol Device:C
- added R4: 4K7, Resistor_THT:R_Axial_DIN0207_L6.3mm_D2.5mm_P10.16mm_Horizontal, symbol Device:R
- added SW2: SW_DIP_x04, Button_Switch_THT:SW_DIP_SPSTx04_Slide_6.7x11.72mm_W7.62mm_P2.54mm_LowProfile, symbol Switch:SW_DIP_x04
- added U3: 74LS157, Package_DIP:DIP-16_W7.62mm, symbol 74xx:74LS157
Connections:
- net +5V: now also C3.1, SW2.1, SW2.2, SW2.3, SW2.4, U3.16 (VCC); no longer R1.2, R2.2, R3.2
- net GND: now also R1.2, R2.2, R3.2, C3.2, R4.2, U3.10 (I1c), U3.11 (I0c), U3.13 (I1d), U3.14 (I0d), U3.15 (E), U3.3 (I1a), U3.8 (GND)
- net at R3.1, U1.1 (A15): now also SW2.8
- net at U1.26 (A13): now also U3.7 (Zb); no longer R1.1
- net at R2.1, U1.27 (A14): now also SW2.7
- net A13: no longer names the net of U2.1 (A0)
- net A13: now also U3.4 (Za); no longer J1.A15 (A13)
- new net: R4.1, SW2.5, U3.1 (S)
- new net: R1.1, SW2.6, U3.5 (I0b)
- new net: J1.A15 (A13), U3.2 (I0a), U3.6 (I1b)
Other:
- moved on the sheet: C1, C2, R1, R2, R3, U1, U2
